Commit message: debug

File: src/omni_description/urdf/wheels.xacro (robot description, xacro)
@@ -18,4 +18,5 @@
       <parent link="${parent}"/><child link="roller_link_${suffix}"/>
       <origin xyz="${xyz}" rpy="${rpy}"/><axis xyz="0 0 1"/>
+      <dynamics damping="0.001" friction="0.001"/>
     </joint>
     <gazebo reference="roller_link_${suffix}">
@@ -29,7 +30,4 @@
         <mesh filename="package://omni_description/meshes/4w/omni_frame.stl"/>
       </geometry><material name="white"><color rgba="1 1 1 1"/></material></visual>
-      <collision><geometry>
-        <mesh filename="package://omni_description/meshes/4w/omni_frame.stl"/>
-      </geometry></collision>
       <inertial><mass value="0.5"/>
         <inertia ixx="0.005" ixy="0" ixz="0" iyy="0.005" iyz="0" izz="0.005"/>
