Commit message: plan

File: src/omni_description/urdf/chassis.xacro (robot description, xacro)
@@ -16,5 +16,5 @@
     </link>
     <joint name="base_joint" type="fixed">
-      <parent link="${parent}"/><child link="base_link"/>
+      <parent link="base_link"/><child link="${parent}"/>
       <origin xyz="0 0 0" rpy="0 0 0"/>
     </joint>

File: src/omni_description/urdf/sensors.xacro (robot description, xacro)
@@ -65,4 +65,16 @@
       </sensor>
     </gazebo>
+    <!-- Canonical alias for laser_link -->
+    <link name="laser_link"/>
+    <joint name="laser_link_alias" type="fixed">
+      <parent link="lidar_link_1"/><child link="laser_link"/>
+      <origin xyz="0 0 0" rpy="0 0 0"/>
+    </joint>
+    <!-- Canonical alias for imu_link -->
+    <link name="imu_link"/>
+    <joint name="imu_link_alias" type="fixed">
+      <parent link="imu_link_1"/><child link="imu_link"/>
+      <origin xyz="0 0 0" rpy="0 0 0"/>
+    </joint>
   </xacro:macro>
 </robot>

Commit message: update agents

File: src/omni_description/urdf/chassis.xacro (robot description, xacro)
@@ -16,5 +16,5 @@
     </link>
     <joint name="base_joint" type="fixed">
-      <parent link="base_link"/><child link="${parent}"/>
+      <parent link="${parent}"/><child link="base_link"/>
       <origin xyz="0 0 0" rpy="0 0 0"/>
     </joint>

File: src/omni_description/urdf/sensors.xacro (robot description, xacro)
@@ -35,5 +35,5 @@
       <!-- Gazebo Harmonic updates lidar through the rendering sensor system;
            keep the supported GPU sensor in both visual and headless profiles. -->
-      <sensor name="gpu_lidar" type="gpu_lidar"><topic>/scan</topic><update_rate>5</update_rate><gz_frame_id>lidar_link_1</gz_frame_id>
+      <sensor name="gpu_lidar" type="gpu_lidar"><topic>/scan</topic><update_rate>10</update_rate><gz_frame_id>lidar_link_1</gz_frame_id>
         <lidar><scan><horizontal><samples>360</samples><resolution>1</resolution><min_angle>-3.1415</min_angle><max_angle>3.1415</max_angle></horizontal></scan>
           <range><min>0.08</min><max>10.0</max><resolution>0.01</resolution></range><noise><type>gaussian</type><mean>0.0</mean><stddev>0.01</stddev></noise>
@@ -53,12 +53,12 @@
         <imu>
           <angular_velocity>
-            <x><noise type="gaussian"><mean>0.0</mean><stddev>0.005</stddev><bias_mean>0.015</bias_mean><bias_stddev>0.0002</bias_stddev></noise></x>
-            <y><noise type="gaussian"><mean>0.0</mean><stddev>0.005</stddev><bias_mean>-0.020</bias_mean><bias_stddev>0.0002</bias_stddev></noise></y>
-            <z><noise type="gaussian"><mean>0.0</mean><stddev>0.005</stddev><bias_mean>0.025</bias_mean><bias_stddev>0.0002</bias_stddev></noise></z>
+            <x><noise type="gaussian"><mean>0.0</mean><stddev>0.0015</stddev><bias_mean>0.003</bias_mean><bias_stddev>0.00005</bias_stddev></noise></x>
+            <y><noise type="gaussian"><mean>0.0</mean><stddev>0.0015</stddev><bias_mean>-0.004</bias_mean><bias_stddev>0.00005</bias_stddev></noise></y>
+            <z><noise type="gaussian"><mean>0.0</mean><stddev>0.0015</stddev><bias_mean>0.004</bias_mean><bias_stddev>0.00005</bias_stddev></noise></z>
           </angular_velocity>
           <linear_acceleration>
-            <x><noise type="gaussian"><mean>0.0</mean><stddev>0.05</stddev><bias_mean>0.12</bias_mean><bias_stddev>0.005</bias_stddev></noise></x>
-            <y><noise type="gaussian"><mean>0.0</mean><stddev>0.05</stddev><bias_mean>-0.18</bias_mean><bias_stddev>0.005</bias_stddev></noise></y>
-            <z><noise type="gaussian"><mean>0.0</mean><stddev>0.05</stddev><bias_mean>0.25</bias_mean><bias_stddev>0.005</bias_stddev></noise></z>
+            <x><noise type="gaussian"><mean>0.0</mean><stddev>0.015</stddev><bias_mean>0.02</bias_mean><bias_stddev>0.001</bias_stddev></noise></x>
+            <y><noise type="gaussian"><mean>0.0</mean><stddev>0.015</stddev><bias_mean>-0.03</bias_mean><bias_stddev>0.001</bias_stddev></noise></y>
+            <z><noise type="gaussian"><mean>0.0</mean><stddev>0.015</stddev><bias_mean>0.04</bias_mean><bias_stddev>0.001</bias_stddev></noise></z>
           </linear_acceleration>
         </imu>

File: src/omni_description/urdf/wheels.xacro (robot description, xacro)
@@ -20,5 +20,5 @@
     </joint>
     <gazebo reference="roller_link_${suffix}">
-      <selfCollide>true</selfCollide>
+      <selfCollide>false</selfCollide>
       <collision><surface><friction><ode><mu>1.0</mu><mu2>1.0</mu2></ode></friction></surface></collision>
     </gazebo>

Commit message: config script and review and system

File: src/omni_description/urdf/chassis.xacro (robot description, xacro)
@@ -12,5 +12,5 @@
       <inertial>
         <mass value="3.0"/>
-        <inertia ixx="0.9" ixy="0.0" ixz="0.0" iyy="0.9" iyz="0.0" izz="0.01"/>
+        <inertia ixx="0.025" ixy="0.0" ixz="0.0" iyy="0.025" iyz="0.0" izz="0.034"/>
       </inertial>
     </link>

Commit message: config topic

File: src/omni_description/urdf/chassis.xacro (robot description, xacro)
@@ -7,9 +7,13 @@
         <mesh filename="package://omni_description/meshes/4w/base_link.dae"/>
       </geometry></visual>
-      <collision><geometry>
-        <mesh filename="package://omni_description/meshes/4w/base_link.stl"/>
-      </geometry></collision>
+      <collision>
+        <origin xyz="0 0 0.0455" rpy="0 0 0"/>
+        <geometry>
+          <box size="0.25 0.25 0.091"/>
+        </geometry>
+      </collision>
       <inertial>
-        <mass value="3.0"/>
+        <origin xyz="0 0 0.02" rpy="0 0 0"/>
+        <mass value="3.5"/>
         <inertia ixx="0.025" ixy="0.0" ixz="0.0" iyy="0.025" iyz="0.0" izz="0.034"/>
       </inertial>
@@ -19,4 +23,7 @@
       <origin xyz="0 0 0" rpy="0 0 0"/>
     </joint>
+    <gazebo reference="base_link">
+      <selfCollide>false</selfCollide>
+    </gazebo>
   </xacro:macro>
 </robot>

File: src/omni_description/urdf/wheels.xacro (robot description, xacro)
@@ -8,7 +8,25 @@
         <mesh filename="package://omni_description/meshes/4w/roller.stl"/>
       </geometry><material name="black"><color rgba="0 0 0 1"/></material></visual>
-      <collision><geometry>
-        <mesh filename="package://omni_description/meshes/4w/roller.stl"/>
-      </geometry></collision>
+      <!-- 5-sphere barrel contour: eliminates 5.7mm polygon cam runout down to <0.04mm for buttery-smooth motion -->
+      <collision name="c0">
+        <origin xyz="0 0 0" rpy="0 0 0"/>
+        <geometry><sphere radius="0.009"/></geometry>
+      </collision>
+      <collision name="c1_pos">
+        <origin xyz="0 0 0.007" rpy="0 0 0"/>
+        <geometry><sphere radius="0.0079"/></geometry>
+      </collision>
+      <collision name="c1_neg">
+        <origin xyz="0 0 -0.007" rpy="0 0 0"/>
+        <geometry><sphere radius="0.0079"/></geometry>
+      </collision>
+      <collision name="c2_pos">
+        <origin xyz="0 0 0.013" rpy="0 0 0"/>
+        <geometry><sphere radius="0.0053"/></geometry>
+      </collision>
+      <collision name="c2_neg">
+        <origin xyz="0 0 -0.013" rpy="0 0 0"/>
+        <geometry><sphere radius="0.0053"/></geometry>
+      </collision>
       <inertial><mass value="0.009"/>
         <inertia ixx="1e-6" ixy="0" ixz="0" iyy="1e-6" iyz="0" izz="1e-6"/>
@@ -18,9 +36,25 @@
       <parent link="${parent}"/><child link="roller_link_${suffix}"/>
       <origin xyz="${xyz}" rpy="${rpy}"/><axis xyz="0 0 1"/>
-      <dynamics damping="0.001" friction="0.001"/>
+      <dynamics damping="0.0001" friction="0.0001"/>
     </joint>
     <gazebo reference="roller_link_${suffix}">
       <selfCollide>false</selfCollide>
-      <collision><surface><friction><ode><mu>1.0</mu><mu2>1.0</mu2></ode></friction></surface></collision>
+      <collision>
+        <surface>
+          <friction>
+            <ode>
+              <mu>1.2</mu>
+              <mu2>1.2</mu2>
+            </ode>
+          </friction>
+          <contact>
+            <ode>
+              <kp>100000.0</kp>
+              <kd>100.0</kd>
+              <min_depth>0.0005</min_depth>
+            </ode>
+          </contact>
+        </surface>
+      </collision>
     </gazebo>
   </xacro:macro>
@@ -30,6 +64,8 @@
         <mesh filename="package://omni_description/meshes/4w/omni_frame.stl"/>
       </geometry><material name="white"><color rgba="1 1 1 1"/></material></visual>
-      <inertial><mass value="0.5"/>
-        <inertia ixx="0.005" ixy="0" ixz="0" iyy="0.005" iyz="0" izz="0.005"/>
+      <inertial>
+        <origin xyz="0 0 0.01" rpy="0 0 0"/>
+        <mass value="0.25"/>
+        <inertia ixx="0.0001" ixy="0" ixz="0" iyy="0.0001" iyz="0" izz="0.00015"/>
       </inertial>
     </link>
@@ -37,7 +73,8 @@
       <parent link="${parent}"/><child link="omni_wheel_link_${suffix}"/>
       <origin xyz="${xyz}" rpy="${rpy}"/><axis xyz="0 0 -1"/>
+      <dynamics damping="0.01" friction="0.01"/>
     </joint>
     <xacro:roller parent="omni_wheel_link_${suffix}" suffix="${suffix}1" xyz="0.0000 -0.0210 0.0175" rpy="-1.570796327 0 -1.570796327"/>
-    <xacro:roller parent="omni_wheel_link_${suffix}" suffix="${suffix}2" xyz="0.0182 0.0105 0.01755" rpy="-1.570796327 0 0.523598776"/>
+    <xacro:roller parent="omni_wheel_link_${suffix}" suffix="${suffix}2" xyz="0.0182 0.0105 0.0175" rpy="-1.570796327 0 0.523598776"/>
     <xacro:roller parent="omni_wheel_link_${suffix}" suffix="${suffix}3" xyz="-0.0182 0.0105 0.0175" rpy="-1.570796327 0 2.617993878"/>
     <xacro:roller parent="omni_wheel_link_${suffix}" suffix="${suffix}4" xyz="-0.0182 -0.0105 0.0025" rpy="-1.570796327 0 -2.617993878"/>
